Commit message: edit urdf to add gripper

File: ur_description/urdf/ur_macro.xacro (robot description, xacro)
@@ -322,19 +322,36 @@
       <child link="${prefix}base"/>
     </joint>
-    <!-- ROS-Industrial 'flange' frame - attachment point for EEF models -->
-    <link name="${prefix}flange" />
-    <joint name="${prefix}wrist_3-flange" type="fixed">
-      <parent link="${prefix}wrist_3_link" />
-      <child link="${prefix}flange" />
-      <origin xyz="0 0 0" rpy="0 ${-pi/2.0} ${-pi/2.0}" />
-    </joint>
-    <!-- ROS-Industrial 'tool0' frame - all-zeros tool frame -->
-    <link name="${prefix}tool0"/>
-    <joint name="${prefix}flange-tool0" type="fixed">
-      <!-- default toolframe - X+ left, Y+ up, Z+ front -->
-      <origin xyz="0 0 0" rpy="${pi/2.0} 0 ${pi/2.0}"/>
-      <parent link="${prefix}flange"/>
-      <child link="${prefix}tool0"/>
-    </joint>
+    <!-- FIXME quick hardcode to mimic ee_link rel pos with waist-->
+    <joint name="ee_fixed_joint" type="fixed">
+        <parent link="wrist_3_link"/>
+        <child link="tool0"/>
+        <origin rpy="0.0 3.141592654 0.0" xyz="0.0 0.0 0.10"/>
+    </joint>
+    <link name="tool0">
+        <collision>
+            <geometry>
+            <box size="0.01 0.01 0.1"/>
+            </geometry>
+            <origin rpy="0 0 0" xyz="-0.08 0 0.05"/>
+        </collision>
+        <visual>
+            <geometry>
+            <box size="0.01 0.01 0.1"/>
+            </geometry>
+            <origin rpy="0 0 0" xyz="-0.08 0 0.05"/>
+        </visual>
+        <collision>
+            <geometry>
+            <box size="0.01 0.01 0.1"/>
+            </geometry>
+            <origin rpy="0 0 0" xyz="0.08 0 0.05"/>
+        </collision>
+        <visual>
+            <geometry>
+            <box size="0.01 0.01 0.1"/>
+            </geometry>
+            <origin rpy="0 0 0" xyz="0.08 0 0.05"/>
+        </visual>
+    </link>
   </xacro:macro>
 </robot>

Commit message: update gripper geometry

File: ur_description/urdf/ur_macro.xacro (robot description, xacro)
@@ -326,30 +326,57 @@
         <parent link="wrist_3_link"/>
         <child link="tool0"/>
-        <origin rpy="0.0 3.141592654 0.0" xyz="0.0 0.0 0.10"/>
+        <origin rpy="0.0 ${pi} ${pi/4}" xyz="0.0 0.0 0.19"/>
     </joint>
     <link name="tool0">
+        <!-- 3D print cylinder -->
         <collision>
             <geometry>
-            <box size="0.01 0.01 0.1"/>
-            </geometry>
-            <origin rpy="0 0 0" xyz="-0.08 0 0.05"/>
+              <cylinder radius="0.05" length="0.04"/>
+            </geometry>
+            <origin rpy="0 0 0" xyz="0.0 0.0 0.17"/>
         </collision>
         <visual>
             <geometry>
-            <box size="0.01 0.01 0.1"/>
-            </geometry>
-            <origin rpy="0 0 0" xyz="-0.08 0 0.05"/>
+              <cylinder radius="0.05" length="0.04"/>
+            </geometry>
+            <origin rpy="0 0 0" xyz="0.0 0.0 0.17"/>
+        </visual>
+        <!-- romo gripper box -->
+        <collision>
+            <geometry>
+              <box size="0.11 0.035 0.08"/>
+            </geometry>
+            <origin rpy="0 0 0" xyz="0.0 0.0 0.11"/>
+        </collision>
+        <visual>
+            <geometry>
+              <box size="0.11 0.035 0.08"/>
+            </geometry>
+            <origin rpy="0 0 0" xyz="0.0 0.0 0.11"/>
+        </visual>
+        <!-- 3D print fingers-->
+        <collision>
+            <geometry>
+            <box size="0.005 0.01 0.07"/>
+            </geometry>
+            <origin rpy="0 0 0" xyz="-0.075 0 0.035"/>
+        </collision>
+        <visual>
+            <geometry>
+            <box size="0.005 0.01 0.07"/>
+            </geometry>
+            <origin rpy="0 0 0" xyz="-0.075 0 0.035"/>
         </visual>
         <collision>
             <geometry>
-            <box size="0.01 0.01 0.1"/>
-            </geometry>
-            <origin rpy="0 0 0" xyz="0.08 0 0.05"/>
+            <box size="0.005 0.01 0.07"/>
+            </geometry>
+            <origin rpy="0 0 0" xyz="0.075 0 0.035"/>
         </collision>
         <visual>
             <geometry>
-            <box size="0.01 0.01 0.1"/>
-            </geometry>
-            <origin rpy="0 0 0" xyz="0.08 0 0.05"/>
+            <box size="0.005 0.01 0.07"/>
+            </geometry>
+            <origin rpy="0 0 0" xyz="0.075 0 0.035"/>
         </visual>
     </link>
